Commit message: merge with latest internal Gitlab version
Signed-off-by: Wolfgang Wiedmeyer <wolfgang.wiedmeyer@kit.edu>

File: urdf/planning_env.urdf.xacro (robot description, xacro)
@@ -5,11 +5,11 @@
   <xacro:arg name="robot_name" default="iiwa"/>
   <xacro:rll_cell hardware_interface="$(arg hardware_interface)" robot_name="$(arg robot_name)"/>
-  <!-- Inser the Maze -->
-  <joint name="Maze" type="fixed">
+  <!-- Insert the maze -->
+  <joint name="maze" type="fixed">
     <parent link="world" />
-    <child link="Maze" />
+    <child link="maze" />
     <origin xyz="0 0 0" rpy="0 0 0"/>
   </joint>
-  <link name="Maze">
+  <link name="maze">
     <inertial>
       <origin xyz="0 0 0" rpy="0 0 0"/>
@@ -23,4 +23,10 @@
       </geometry>
     </visual>
+    <collision>
+      <origin xyz="0 0 0" rpy="0 0 0"/>
+      <geometry>
+        <mesh filename="package://rll_planning_project/meshes/collision/Maze.stl" />
+      </geometry>
+    </collision>
   </link>
 </robot>

Commit message: urdf: attach maze to table
Then it has the same physical properties as the table.

Closes #23

Signed-off-by: Wolfgang Wiedmeyer <wolfgang.wiedmeyer@kit.edu>

File: urdf/planning_env.urdf.xacro (robot description, xacro)
@@ -7,5 +7,5 @@
   <!-- Insert the maze -->
   <joint name="maze" type="fixed">
-    <parent link="world" />
+    <parent link="table" />
     <child link="maze" />
     <origin xyz="0 0 0" rpy="0 0 0"/>
